File: rp2040_example/rp2040_example.kicad_sch (KiCad schematic)
At the start: 20 parts, among them J1 USB_B_Micro, J2 Conn_02x06_Odd_Even, SW1 SW_Omron_B3FS, U1 RP2040, U2 NCP1117-3.3_SOT223, U3 W25Q128JVS, Y1 ABM8-272-T3

Commit message: Change reference on RP2040 example
Parts:
- renumbered D101 to D1
Changed lines of the file:
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@@
   (symbol (lib_id "Device:LED_RBGA") (at 127 161.29 0) (unit 1)
     (in_bom yes) (on_board yes) (dnp no) (fields_autoplaced)
-    (property "Reference" "D101" (at 127 148.59 0)
+    (property "Reference" "D1" (at 127 148.59 0)
       (effects (font (size 1.27 1.27)))
     )
@@
       (project "rp2040_example"
         (path "/16c5b016-7c52-4f61-96e2-bedcca5aba58"
-          (reference "D101") (unit 1)
+          (reference "D1") (unit 1)
         )
       )
