File: handheld/handheld.kicad_pcb (KiCad board)
At the start: 6 copper layers, 103 parts, among them J101 DNP, J102 DNP, J103 Conn_02x05_Odd_Even, J104 Conn_01x02, J105 Conn_02x03_Odd_Even, P101 USB_C_Plug_USB2.0, Q101 AO3401A, Q102 AO3401A, SW101 SW_Omron_B3FS, SW102 SW_SPDT, SW103 SW_Push, SW104 SW_Push, SW105 SW_Push, SW106 SW_Push, SW107 SW_Push, SW108 SW_Push, SW109 SW_Omron_B3FS, SW110 SW_SPDT, SW111 SW_Push, SW112 SW_Push, SW113 SW_Push, SW114 SW_Push, U101 LTC4054ES5-4.2, U102 W25Q128JVS, U103 RP2040, U104 TLV62568DDC, U105 TLV62568DDC, U106 4051, U107 PAM8301, U108 LM321, U109 ESP32-WROVER-E, U110 10k Pot Joystick, U111 10k Pot Joystick, U112 XC6206PxxxMR, Y101 ABM8-272-T3

Commit message: Sent off a version
Parts:
- added C117: 1u, Capacitor_SMD:C_0402_1005Metric, F.Cu at (62.0, 65.9)
- added H101: MountingHole_Pad, MountingHole:MountingHole_3.2mm_M3_DIN965_Pad, F.Cu at (40.0, 40.0)
- added H102: MountingHole_Pad, MountingHole:MountingHole_3.2mm_M3_DIN965_Pad, F.Cu at (130.0, 100.1)
- added H103: MountingHole_Pad, MountingHole:MountingHole_3.2mm_M3_DIN965_Pad, F.Cu at (80.0, 139.9)
- added Q103: AO3401A, Package_TO_SOT_SMD:SOT-23, F.Cu at (52.6, 58.2)
- SW113, SW114: footprint symbols:ALPSALPINE_SKPMBHE010 -> symbols:Horizontal_Button_TS24CA
- U110, U111: footprint Connector_PinHeader_2.54mm:PinHeader_1x04_P2.54mm_Vertical -> symbols:Flat_Analog_Stick
- moved C115 147.8 mm to (53.4, 117.4)
- moved U109 147.4 mm to (42.0, 109.1)
- moved J102 147.3 mm to (55.3, 102.4)
- moved C114 147.2 mm to (53.5, 120.4)
- moved R130 144.3 mm to (56.4, 118.8), turned to 0 degrees
- moved TP105 136.4 mm to (56.7, 130.1), turned to 0 degrees
- moved Q101 130.8 mm to (59.4, 117.5)
- moved R132 130.8 mm to (58.5, 114.5)
- moved R137 130.8 mm to (60.7, 114.6)
- moved SW102 130.8 mm to (61.3, 124.0)
- moved U112 130.8 mm to (55.8, 125.0)
- moved SW109 129.4 mm to (46.0, 86.7), turned to 0 degrees
- moved D102 124.5 mm to (54.7, 116.3), turned to -90 degrees
- moved R128 123.8 mm to (54.6, 114.1), turned to 90 degrees
- moved J101 107.1 mm to (71.5, 127.3), turned to 90 degrees
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Connections:
- J103 pad 6: /LCD_LED -> Net-(J103-Pin_6)
- R128 pad 2: Net-(U109-IO21) -> Net-(U109-IO35)
- U109 pad 33: Net-(U109-IO21) -> unconnected-(U109-IO21-Pad33)
- U109 pad 7: unconnected-(U109-IO35-Pad7) -> Net-(U109-IO35)
Routing:
- net /BUTTON8: track 0.00 -> 118.9 mm, vias 0 -> 2
- net /WL_UART_MISO: track 0.00 -> 106.9 mm, vias 0 -> 3
- net /WL_UART_MOSI: track 0.00 -> 98.2 mm, vias 0 -> 3
- net /STICK0_Y: track 0.00 -> 86.5 mm, vias 0 -> 1
- net /STICK0_X: track 0.00 -> 83.4 mm, vias 0 -> 1
- net /BUTTON4: track 0.00 -> 73.6 mm, vias 0 -> 2
- net /BUTTON6: track 0.00 -> 73.1 mm, vias 0 -> 2
- net /STICK1_X: track 0.00 -> 70.8 mm, vias 0 -> 2
- net /STICK1_Y: track 0.00 -> 68.0 mm, vias 0 -> 2
- net /WL_EN: track 2.64 -> 61.1 mm, vias 0 -> 3
- net /BUTTON7: track 0.00 -> 58.3 mm, vias 0 -> 2
- net /BUTTON5: track 0.00 -> 55.5 mm, vias 0 -> 2
- net /BUTTON0: track 0.00 -> 51.3 mm, vias 0 -> 2
- net /BUTTON9: track 0.00 -> 49.1 mm, vias 0 -> 2
- net /WL_POWER_~{EN}: track 0.00 -> 48.1 mm, vias 0 -> 2
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Other:
- board outline added: 106.8 x 130.8 mm
- board text added: "<MAIN | UART>"
- board text added: "BOOTSEL"
- board text added: "CHRG"
- board text added: "WL BOOT"
- board text added: "WL_JTAG_TMS WL_JTAG_TDI WL_JTAG_TCK WL_JTAG_TDO"
- board text added: "WL_UART_5V WL_UART_MOSI WL_UART_MISO GND"
