File: handheld/handheld.kicad_sch (KiCad schematic)
At the start: 71 parts, among them P101 USB_C_Plug_USB2.0, SW1 SW_Omron_B3FS, SW102 SW_SPST, SW103 SW_Push, SW104 SW_Push, SW105 SW_Push, SW106 SW_Push, SW107 SW_Push, SW108 SW_Push, SW109 SW_Push, SW110 SW_Push, U1 RP2040, U101 LTC4054ES5-4.2, U102 TLV62568DDC, U106 4051, U106 TLV62568DDC, U107 PAM8301, U108 LM321, U3 W25Q128JVS, Y1 ABM8-272-T3

Commit message: More changes
Parts:
- added R4: 10k, Resistor_SMD:R_0402_1005Metric, symbol Device:R
- added R4: 100k, Resistor_SMD:R_0402_1005Metric, symbol Device:R
- R4: value 47k -> 68k
Connections:
- net +3V3: no longer R4.2
- net GND: now also R4.1
- net VBUS: now also R4.2
- net ~{CHRG}: now also R4.1; no longer R4.1, U1.6 (GPIO4)
- net 3V3PG renamed 3V3_GOOD
- new net: R4.1, R4.2, R4.2, U1.6 (GPIO4)
Other:
- moved on the sheet: R3, R4

Commit message: More nonsense
Parts:
- removed R4 (x2): 47k, Resistor_SMD:R_0402_1005Metric, symbol Device:R
- removed R4: 68k, Resistor_SMD:R_0402_1005Metric, symbol Device:R
- removed SW102: SW_SPST, symbol Switch:SW_SPST
- removed SW109, SW110: SW_Push, symbol Switch:SW_Push
- added C115: 100n, Capacitor_SMD:C_0402_1005Metric, symbol Device:C
- added C115: 22u, Capacitor_SMD:C_0603_1608Metric, symbol Device:C
- added C2: 1u, Capacitor_SMD:C_0402_1005Metric, symbol Device:C
- added D105 (x3): LED, LED_SMD:LED_0402_1005Metric, symbol Device:LED
- added F101: I_{hold}=1A, I_{trip}=2A, R_{1max}=0.27Ω, Fuse:Fuse_0805_2012Metric, symbol Device:Fuse
- added J101, J102: DNP, Connector_PinHeader_2.54mm:PinHeader_1x04_P2.54mm_Vertical, symbol Connector_Generic:Conn_01x04
- added J103: Conn_02x05_Odd_Even, Connector_PinHeader_2.54mm:PinHeader_2x05_P2.54mm_Vertical, symbol Connector_Generic:Conn_02x05_Odd_Even
- added J104: Conn_01x02, Connector_PinHeader_2.54mm:PinHeader_1x02_P2.54mm_Vertical, symbol Connector_Generic:Conn_01x02
- added J105: Conn_02x03_Odd_Even, symbols:02x03_Edge_Board_Connector_ER06BGFBK, symbol Connector_Generic:Conn_02x03_Odd_Even
- added Q101, Q102: AO3401A, Package_TO_SOT_SMD:SOT-23, symbol Transistor_FET:AO3401A
- added R4 (x6): 47k, Resistor_SMD:R_0402_1005Metric, symbol Device:R
- added R4: 470, Resistor_SMD:R_0402_1005Metric, symbol Device:R
- added R4 (x3): 220, Resistor_SMD:R_0402_1005Metric, symbol Device:R
- added SW1: SW_Omron_B3FS, Button_Switch_THT:SW_PUSH_6mm, symbol Switch:SW_Omron_B3FS
- added SW102, SW110: SW_SPDT, symbols:MK-12C02-G025_Slide_Switch, symbol Switch:SW_SPDT
- added SW111, SW112, SW113, SW114: SW_Push, symbols:ALPSALPINE_SKPMBHE010, symbol Switch:SW_Push
- added TP106: ESP32-3.3v, TestPoint:TestPoint_THTPad_D1.0mm_Drill0.5mm, symbol Connector:TestPoint
- added U109: ESP32-WROVER-E, symbols:ESP32-WROVER-IE, symbol CustomSymbols:ESP32-WROVER-E
- added U110, U111: 10k Pot Joystick, Connector_PinHeader_2.54mm:PinHeader_1x04_P2.54mm_Vertical, symbol CustomSymbols:Dual_Potentiometer_Joystick
- added U112: XC6206PxxxMR, Package_TO_SOT_SMD:SOT-23-3, symbol Regulator_Linear:XC6206PxxxMR
- BT101, RV101: footprint (none) -> Connector_PinHeader_2.54mm:PinHeader_1x02_P2.54mm_Vertical
- C113, C114, C115, C116: footprint Capacitor_SMD:C_0805_2012Metric -> Capacitor_SMD:C_0603_1608Metric
- D1: LCSC (none) -> C458749
- P101: footprint (none) -> Connector_USB:USB_C_Receptacle_G-Switch_GT-USB-7010ASV; LCSC (none) -> C2988369
- R101, R102: footprint (none) -> Resistor_SMD:R_0402_1005Metric
- R114, R115, R116, R117: footprint Resistor_SMD:R_0805_2012Metric -> Resistor_SMD:R_0402_1005Metric
- R3, R4: value 100k -> 47k
- R4: value 10k -> 47k
- SW1: LCSC (none) -> C493038
- SW103, SW104, SW105, SW106, SW107, SW108: footprint (none) -> symbols:ALPSALPINE_SKPMBHE010; LCSC (none) -> C115350
- U1: LCSC (none) -> C2040
- U101: LCSC (none) -> C462648
- U102, U106: LCSC (none) -> C2071019
- U106: footprint (none) -> Package_SO:SOP-16_3.9x9.9mm_P1.27mm; LCSC (none) -> C2943297
- U107: LCSC (none) -> C3001605
- U108: LCSC (none) -> C5252901
- U3: LCSC (none) -> C97521
- Y1: LCSC (none) -> C70565
Connections:
- net +3V3: now also R4.1, C2.1, D105.2 (A), D105.2 (A), J103.8 (Pin_8), J105.2 (Pin_2), Q101.2 (S), Q102.2 (S), R4.2, SW111.2, SW112.2, SW113.2, SW114.2, U110.4 (PWR), U111.4 (PWR)
- net +3V8: now also SW110.2 (B)
- net +BATT: now also F101.2, SW110.1 (A); no longer BT101.1 (+)
- net ADC_MUX_S0: now also U1.39 (GPIO27_ADC1)
- net ADC_MUX_S1: now also U1.40 (GPIO28_ADC2)
- net ADC_MUX_S2: now also U1.41 (GPIO29_ADC3)
- net AUDIO_EN: now also U1.15 (GPIO12); no longer U1.8 (GPIO6)
- net AUDIO_OUT: now also U1.14 (GPIO11); no longer U1.7 (GPIO5)
- net BATT_SENSE: now also U106.1 (X4); no longer U1.38 (GPIO26_ADC0)
- net BUTTON0: now also U1.7 (GPIO5); no longer U1.9 (GPIO7)
- net BUTTON1: now also U1.8 (GPIO6); no longer U1.11 (GPIO8)
- net BUTTON2: now also U1.9 (GPIO7); no longer U1.12 (GPIO9)
- net BUTTON3: now also U1.11 (GPIO8); no longer U1.13 (GPIO10)
- net BUTTON4: now also U1.12 (GPIO9); no longer U1.14 (GPIO11)
- net BUTTON5: now also U1.13 (GPIO10); no longer U1.15 (GPIO12)
- net BUTTON6: now also R4.2, SW111.1
- net BUTTON7: now also R4.2, SW112.1
- net GND: now also C115.2, C115.2, C2.2, J101.4 (Pin_4), J103.10 (Pin_10), J103.9 (Pin_9), J105.5 (Pin_5), R4.1, R4.1, R4.1, R4.1, SW1.2, U109.1 (GND), U109.15 (GND), U109.38 (GND), U109.39 (GND_BOTTOM), U110.2 (GND), U111.2 (GND), U112.1 (GND)
- net LCD_SPI_CLK: now also J103.3 (Pin_3)
- net LCD_SPI_CS: now also J103.5 (Pin_5)
- net LCD_SPI_MISO: now also J103.7 (Pin_7)
- net LCD_SPI_MOSI: now also J103.1 (Pin_1)
- net MUXED_ADC: now also U1.38 (GPIO26_ADC0); no longer U1.40 (GPIO28_ADC2)
- net SPEAKER+: now also J104.1 (Pin_1)
- net SPEAKER-: now also J104.2 (Pin_2)
- net STICK0_X: now also U110.1 (LeftRight)
- net STICK0_Y: now also U110.3 (UpDown)
- net STICK1_X: now also U111.1 (LeftRight)
- net STICK1_Y: now also U111.3 (UpDown)
- net USB_D+: now also R3.2; no longer R3.1
- net USB_D-: now also R4.2; no longer R4.1
- net VBUS_SENSE: now also U106.5 (X5); no longer U1.39 (GPIO27_ADC1)
- net ~{CHRG}: now also R4.2, Q102.1 (G); no longer R4.1
- net GAME_CART_TX: now reaches U1.18 (GPIO15)
- net GAME_CART_TX: now also J105.3 (Pin_3)
- net GAME_CART_RX: now reaches U1.27 (GPIO16)
- net GAME_CART_RX: now also J105.1 (Pin_1)
- net LCD_DC: now reaches U1.28 (GPIO17)
- net LCD_DC: now also J103.2 (Pin_2)
- net WL_POWER_~{EN}: now reaches U1.29 (GPIO18)
- net WL_POWER_~{EN}: now also R4.2
- net WL_EN: now reaches U1.30 (GPIO19)
- net WL_EN: now also R4.2, U109.3 (EN)
- net WL_UART_MOSI: now reaches U1.31 (GPIO20)
- net WL_UART_MOSI: now also J101.2 (Pin_2), U109.34 (RXD0)
- net WL_UART_MISO: now reaches U1.32 (GPIO21)
- net WL_UART_MISO: now also J101.3 (Pin_3), U109.35 (TXD0)
- net LCD_RESET: now reaches U1.34 (GPIO22)
- net LCD_RESET: now also J103.4 (Pin_4)
- net DBG_LED0: now reaches U1.35 (GPIO23)
- net DBG_LED0: now also R4.2
- net DBG_LED1: now reaches U1.36 (GPIO24)
- net DBG_LED1: now also R4.2
- net LCD_LED: now reaches U1.37 (GPIO25)
- net LCD_LED: now also J103.6 (Pin_6)
- net at U1.46 (USB_DM): now also R4.1; no longer R4.2
- net at U1.47 (USB_DP): now also R3.1; no longer R3.2
- net at R4.2, U1.6 (GPIO4): now also Q102.3 (D); no longer R4.2
- net at R2.2, TP106.1, U108.4: now also RV101.1; no longer RV101.3
- net BUTTON8: now reaches U106.2 (X6)
- net BUTTON8: now also R4.2, SW113.1
- net BUTTON9: now reaches U106.4 (X7)
- net BUTTON9: now also R4.2, SW114.1
- new net: SW1.1, U109.25 (IO0)
- new net: R4.2, U109.33 (IO21)
- new net: BT101.1 (+), F101.1
- new net: D105.1 (K), R4.1 (x3)
- new net: Q101.1 (G), R4.1, R4.1
- new net: SW102.3 (C), U112.2 (VO)
- new net GATED_WL_POWER: Q101.3 (D), SW102.1 (A)
- new net WL_JTAG_TCK: J102.3 (Pin_3), U109.16 (IO13)
- new net WL_JTAG_TDI: J102.2 (Pin_2), U109.14 (IO12)
- new net WL_JTAG_TDO: J102.4 (Pin_4), U109.23 (IO15)
- new net WL_JTAG_TMS: J102.1 (Pin_1), U109.13 (IO14)
- new net WL_POWER: C115.1, C115.1, D105.2 (A), R4.1, SW102.2 (B), TP106.1, U109.2 (3V3)
- new net WL_UART_5V: J101.1 (Pin_1), U112.3 (VI)
- no-connect marks 24 -> 36
Other:
- note added: "Analog Sticks"
- note added: "Charging Indicator"
- note added: "Charging Port/Flashing"
- note added: "D Pad"
- note added: "Debug LEDs"
- note added: "ESP32 Programming"
- note added: "Face Buttons"
- note added: "Game Cart"
- note added: "Hold at power up for boot option"
- note added: "ILI9341 TFT LCD"
- note added: "Keep these resistors close to RP2040"
- note added: "Keep this cap close to pin 44"
- note added: "Keep this cap close to pin 45"
- note added: "Main Power Switch"
- note added: "Shoulder Buttons"
- note added: "This is effectively a PMOS inverter, that level-shifts 5V ~{CHRG} into 3.3V CHRG"
- note added: "Wireless"
- note removed: "Buttons"
- note removed: "Charging Indicators"
- note removed: "Make sure C2 is close to pin 45 of RP2040"
- note removed: "Make sure C3 is close to pin 44 of RP2040"
- note removed: "Make sure R3 and R4 are close to RP2040"
- moved on the sheet: BT101, C113, C114, C115, C116, C2, C3, C4, C5, D1, L101, L102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

Commit message: Sent off a version
Parts:
- added C2: 1u, Capacitor_SMD:C_0402_1005Metric, symbol Device:C
- added H101, H102, H103: MountingHole_Pad, MountingHole:MountingHole_3.2mm_M3_DIN965_Pad, symbol Mechanical:MountingHole_Pad
- added Q103: AO3401A, Package_TO_SOT_SMD:SOT-23, symbol Transistor_FET:AO3401A
- SW113: footprint symbols:ALPSALPINE_SKPMBHE010 -> symbols:Horizontal_Button_TS24CA; LCSC C393942 -> C393942
- SW114: footprint symbols:ALPSALPINE_SKPMBHE010 -> symbols:Horizontal_Button_TS24CA
- U110, U111: footprint Connector_PinHeader_2.54mm:PinHeader_1x04_P2.54mm_Vertical -> symbols:Flat_Analog_Stick
Connections:
- net +1V1: now also C2.1
- net +3V3: now also Q103.2 (S)
- net GND: now also C2.2, H101.1, H102.1, H103.1
- net LCD_LED: now also Q103.1 (G); no longer J103.6 (Pin_6)
- net at U109.33 (IO21): no longer R4.2
- net at U109.7 (IO35): now also R4.2
- new net: J103.6 (Pin_6), Q103.3 (D)
Other:
- note added: "Keep this cap close to pin 23"
- moved on the sheet: D105, R4
