File: artix7-practice/artix7-practice.kicad_sch (KiCad schematic)
At the start: 50 parts, among them J101 USB_B_Micro, J102 Conn_02x06_Odd_Even, Q101 Q_NMOS_GSD, U101 XC7A35T-FTG256, U102 TLV62568DDC, U103 TLV62568DDC, U104 FT2232HL, U105 93CxxC, U106 W25Q128JVS, X101 125MHz, Y101 ABM8-272-T3

Commit message: Final version before switching from XC7A35T-xFTG256 to -xCSG325
Parts:
- removed C101, C102, C103, C104: 22u, Capacitor_SMD:C_0603_1608Metric, symbol Device:C
- removed L101, L102: 2.2uH, Inductor_SMD:L_Taiyo-Yuden_NR-40xx, symbol Device:L
- removed R101: 39k, Resistor_SMD:R_0402_1005Metric, symbol Device:R
- removed R102: 62k, Resistor_SMD:R_0402_1005Metric, symbol Device:R
- removed R103: 68k, Resistor_SMD:R_0402_1005Metric, symbol Device:R
- removed R104: 33k, Resistor_SMD:R_0402_1005Metric, symbol Device:R
- removed U102, U103: TLV62568DDC, Package_TO_SOT_SMD:SOT-23-6, symbol Regulator_Switching:TLV62568DDC
- added C115, C116, C117, C118, C119, C120: 100n, Capacitor_SMD:C_0201_0603Metric, symbol Device:C
- added C121, C125, C129: 100n, Capacitor_SMD:C_0402_1005Metric, symbol Device:C
- added C122, C123, C126, C127, C130, C131: 22u, Capacitor_SMD:C_0805_2012Metric, symbol Device:C
- added C124, C128, C132: 1u, Capacitor_SMD:C_0402_1005Metric, symbol Device:C
- added D101, D108: MBRA340, Diode_SMD:D_SMA, symbol Diode:MBRA340
- added J103: Bus_PCI_Express_x1, Connector_PCBEdge:BUS_PCIexpress_x1, symbol Connector:Bus_PCI_Express_x1
- added L104, L105, L106: 2.2uH, Inductor_SMD:L_Taiyo-Yuden_NR-40xx, symbol Device:L
- added R122, R123: 4.7k, Resistor_SMD:R_0402_1005Metric, symbol Device:R
- added R124: 43k, Resistor_SMD:R_0402_1005Metric, symbol Device:R
- added R125: 56k, Resistor_SMD:R_0402_1005Metric, symbol Device:R
- added R126: 68k, Resistor_SMD:R_0402_1005Metric, symbol Device:R
- added R127: 30k, Resistor_SMD:R_0402_1005Metric, symbol Device:R
- added R128: 1k, Resistor_SMD:R_0402_1005Metric, symbol Device:R
- added R129: 150k, Resistor_SMD:R_0402_1005Metric, symbol Device:R
- added U102: XC7A35T-CSG325, symbol FPGA_Xilinx_Artix7:XC7A35T-CSG325
- added U108, U109, U110: LMR33630ADDA, Package_SO:Texas_HSOP-8-1EP_3.9x4.9mm_P1.27mm_ThermalVias, symbol Regulator_Switching:LMR33630ADDA
- U101: footprint (none) -> easyeda2kicad:FBGA-256_L17.0-W17.0-R16-C16-P1.00-TL; LCSC (none) -> C181716
Connections:
- net +1V0: now also C123.1, L104.2, R128.1
- net +1V8: now also C127.1, L105.2, R124.1
- net +3V3: now also U101.E7 (CFGBVS_0), U101.L9 (PROGRAM_B_0), U101.M9 (M0_0), C131.1, L106.2, R126.1
- net DONE: now also U101.H10 (DONE_0)
- net FLASH_IO0: now also U101.J13 (IO_L1P_T0_D00_MOSI_14)
- net FLASH_IO1: now also U101.J14 (IO_L1N_T0_D01_DIN_14)
- net FLASH_IO2: now also U101.K15 (IO_L2P_T0_D02_14)
- net FLASH_IO3: now also U101.K16 (IO_L2N_T0_D03_14)
- net FLASH_~{CS}: now also U101.L12 (IO_L6P_T0_FCS_B_14)
- net GND: now also U101.H7 (VREFN_0), U101.H8 (VP_0), U101.J7 (VN_0), U101.J8 (VREFP_0), U101.K7 (DXN_0), U101.K8 (DXP_0), U101.M10 (M1_0), U101.M11 (M2_0), C122.2, C123.2, C124.2, C126.2, C127.2, C128.2, C130.2, C131.2, C132.2, J103.A12 (GND), J103.A15 (GND), J103.A18 (GND), J103.A4 (GND), J103.B13 (GND), J103.B16 (GND), J103.B18 (GND), J103.B4 (GND), J103.B7 (GND), R125.2, R127.2, R129.2, U108.1 (GND), U108.9 (GND), U109.1 (GND), U109.9 (GND), U110.1 (GND), U110.9 (GND)
- net +5V renamed VBUS
- net VBUS: now also D108.2 (A)
- new net: R126.2, R127.1, U110.5 (FB)
- new net: C125.1, U109.7 (BOOT)
- new net: C125.2, L105.1, U109.8 (SW)
- new net: C121.2, L104.1, U108.8 (SW)
- new net: C124.1, U108.6 (VCC)
- new net: R124.2, R125.1, U109.5 (FB)
- new net: C118.2, J103.B15 (PETn0)
- new net: U108.4 (PG), U109.3 (EN)
- new net: U109.4 (PG), U110.3 (EN)
- new net: C128.1, U109.6 (VCC)
- new net: C116.2, J103.A14 (REFCLK-)
- new net: C132.1, U110.6 (VCC)
- new net: C129.1, U110.7 (BOOT)
- new net: C129.2, L106.1, U110.8 (SW)
- new net: C120.1, J103.A17 (PERn0)
- new net: C115.2, J103.A13 (REFCLK+)
- new net: C117.2, J103.B14 (PETp0)
- new net: R128.2, R129.1, U108.5 (FB)
- new net: J103.A1 (~{PRSNT1}), J103.B17 (~{PRSNT2})
- new net: J103.A10 (+3.3V), J103.A9 (+3.3V), J103.B8 (+3.3V)
- new net: C119.1, J103.A16 (PERp0)
- new net: C121.1, U108.7 (BOOT)
- new net +12V: D101.2 (A), J103.A2 (+12V), J103.A3 (+12V), J103.B1 (+12V), J103.B2 (+12V), J103.B3 (+12V)
- new net 3V3_AUX: J103.B10 (3.3Vaux), R122.1, R123.1
- new net MAIN_PWR: C122.1, C126.1, C130.1, U108.2 (VIN), U108.3 (EN), U109.2 (VIN), U110.2 (VIN)
- new net PCIE_RX0+: C117.1
- new net PCIE_RX0-: C118.1
- new net PCIE_TX0+: C119.2
- new net PCIE_TX0-: C120.2
- new net PCIE_~{PERST}: J103.A11 (~{PERST}), R123.2
- new net PCIE_~{WAKE}: J103.B11 (~{WAKE}), R122.2
- new net POWER: D101.1 (K), D108.1 (K)
- new net REFCLK+: C115.1
- new net REFCLK-: C116.1
- no-connect marks 33 -> 42
Other:
- note added: "M[2:0] == 001 (Master SPI)"
- note added: "Vout = 1.01"
- note added: "Vout = 1.77"
- note added: "Vout = 3.27"
- note removed: "Vout = 0.98"
- note removed: "Vout = 1.84"
- moved on the sheet: C111, R107, R108, R114, U106

Commit message: JLCPCB uploads
Parts:
- removed U101: XC7A35T-FTG256, easyeda2kicad:FBGA-256_L17.0-W17.0-R16-C16-P1.00-TL, symbol FPGA_Xilinx_Artix7:XC7A35T-FTG256
- added C101: 100n, Capacitor_SMD:C_0402_1005Metric, symbol Device:C
- added C102, C103: 22u, Capacitor_SMD:C_0805_2012Metric, symbol Device:C
- added C104: 1u, Capacitor_SMD:C_0402_1005Metric, symbol Device:C
- added C113, C114, C162, C163, C164, C165: 22u, Capacitor_SMD:C_0603_1608Metric, symbol Device:C
- added C133, C134, C135, C136, C137, C139, C142, C143, C146, C147, C150, C151, C154, C155, C156, C158, C159, C160, C161: 1u, Capacitor_SMD:C_0201_0603Metric, symbol Device:C
- added C138, C140, C141, C144, C145, C148, C149, C152, C153, C157: 100n, Capacitor_SMD:C_0201_0603Metric, symbol Device:C
- added L101, L102, L103: 2.2uH, Inductor_SMD:L_Taiyo-Yuden_NR-40xx, symbol Device:L
- added R101: 18k, Resistor_SMD:R_0402_1005Metric, symbol Device:R
- added R102: 82k, Resistor_SMD:R_0402_1005Metric, symbol Device:R
- added R103: 100, Resistor_SMD:R_0402_1005Metric, symbol Device:R
- added U101: LMR33630ADDA, Package_SO:Texas_HSOP-8-1EP_3.9x4.9mm_P1.27mm_ThermalVias, symbol Regulator_Switching:LMR33630ADDA
- U102: footprint (none) -> Package_BGA:Xilinx_CSG325; LCSC (none) -> C1521749
Connections:
- net POWER is gone; now on net MAIN_PWR: D101.1 (K), D108.1 (K)
- net +1V0: now also U102.F11 (VCCBRAM), U102.F7 (VCCINT), U102.F9 (VCCINT), U102.G10 (VCCBRAM), U102.G8 (VCCINT), U102.H11 (VCCBRAM), U102.H7 (VCCINT), U102.H9 (VCCINT), U102.J12 (VCCINT), U102.J8 (VCCINT), U102.K11 (VCCINT), U102.K7 (VCCINT), U102.L12 (VCCINT), U102.L8 (VCCINT), U102.M11 (VCCINT), U102.M7 (VCCINT), U102.N10 (VCCINT), U102.N12 (VCCINT), U102.N8 (VCCINT), U102.P11 (VCCINT), U102.P9 (VCCINT), C139.1, C143.1, C144.1, C145.1, C146.1, C147.1, C148.1, C149.1, C150.1, C151.1, C152.1, C153.1, L102.1
- net +1V8: now also U102.G12 (VCCAUX), U102.H13 (VCCAUX), U102.J10 (VCCADC_0), U102.K13 (VCCAUX), U102.M13 (VCCAUX), U102.P13 (VCCAUX), C154.1, C155.1, C156.1, C157.1, C158.1
- net +3V3: now also U102.A16 (VCCO_15), U102.B13 (VCCO_15), U102.C10 (VCCO_15), U102.D17 (VCCO_15), U102.E10 (VCCO_0), U102.E12 (CFGBVS_0), U102.E14 (VCCO_15), U102.G18 (VCCO_15), U102.H15 (VCCO_15), U102.L16 (VCCO_14), U102.L6 (VCCO_34), U102.M3 (VCCO_34), U102.P10 (PROGRAM_B_0), U102.P17 (VCCO_14), U102.P7 (VCCO_34), U102.R10 (VCCO_0), U102.R12 (M0_0), U102.R14 (VCCO_14), U102.R4 (VCCO_34), U102.T1 (VCCO_34), U102.T11 (VCCO_14), U102.U18 (VCCO_14), U102.U8 (VCCO_14), U102.V15 (VCCO_14), U102.V5 (VCCO_34), C159.1, C160.1, C161.1, C162.1, C163.1, C164.1, C165.1
- net CLK125MHZ: now also U102.A17 (IO_L15N_T2_DQS_ADV_B_15)
- net DONE: now also U102.F12 (DONE_0)
- net FLASH_CLK: now also U102.E8 (CCLK_0)
- net FLASH_IO0: now also U102.K16 (IO_L1P_T0_D00_MOSI_14)
- net FLASH_IO1: now also U102.L17 (IO_L1N_T0_D01_DIN_14)
- net FLASH_IO2: now also U102.J15 (IO_L2P_T0_D02_14)
- net FLASH_IO3: now also U102.J16 (IO_L2N_T0_D03_14)
- net FLASH_~{CS}: now also U102.L15 (IO_L6P_T0_FCS_B_14)
- net GND: now also U102.A1 (GND), U102.A11 (GND), U102.A18 (GND), U102.A3 (MGTPRXN1_216), U102.A4 (MGTPRXP1_216), U102.A5 (GND), U102.A7 (GND), U102.A8 (GND), U102.B18 (GND), U102.B3 (GND), U102.B5 (MGTREFCLK1N_216), U102.B6 (MGTREFCLK1P_216), U102.B7 (GND), U102.B8 (GND), U102.C15 (GND), U102.C2 (GND), U102.C3 (MGTPRXN2_216), U102.C4 (MGTPRXP2_216), U102.C6 (GND), U102.C7 (GND), U102.D12 (GND), U102.D3 (GND), U102.D4 (GND), U102.D7 (GND), U102.E11 (VCCBATT_0), U102.E2 (GND), U102.E6 (GND), U102.E7 (GND), U102.E9 (GND), U102.F10 (GND), U102.F13 (M2_0), U102.F16 (GND), U102.F4 (GND), U102.F6 (GND), U102.G1 (GND), U102.G11 (GND), U102.G13 (GND), U102.G3 (MGTPRXN3_216), U102.G4 (MGTPRXP3_216), U102.G5 (GND), U102.G6 (GND), U102.G7 (GND), U102.G9 (GND), U102.H10 (GND), U102.H12 (GND), U102.H3 (GND), U102.H4 (GND), U102.H5 (GND), U102.H6 (GND), U102.H8 (GND), U102.J1 (GND), U102.J11 (GND), U102.J13 (GND), U102.J17 (GND), U102.J2 (GND), U102.J3 (GND), U102.J7 (GND), U102.J9 (GNDADC_0), U102.K10 (VP_0), U102.K12 (GND), U102.K14 (GND), U102.K4 (GND), U102.K8 (GND), U102.K9 (VREFN_0), U102.L1 (GND), U102.L10 (VREFP_0), U102.L11 (GND), U102.L13 (GND), U102.L7 (GND), U102.L9 (VN_0), U102.M10 (DXP_0), U102.M12 (GND), U102.M18 (GND), U102.M8 (GND), U102.M9 (DXN_0), U102.N11 (GND), U102.N13 (GND), U102.N15 (GND), U102.N5 (GND), U102.N7 (GND), U102.N9 (GND), U102.P12 (GND), U102.P2 (GND), U102.P8 (GND), U102.R11 (M1_0), U102.R9 (GND), U102.T16 (GND), U102.T6 (GND), U102.U13 (GND), U102.U3 (GND), U102.V1 (GND), U102.V10 (GND), U102.V18 (GND), C102.2, C103.2, C104.2, C113.2, C114.2, C133.2, C134.2, C135.2, C136.2, C137.2, C138.2, C139.2, C140.2, C141.2, C142.2, C143.2, C144.2, C145.2, C146.2, C147.2, C148.2, C149.2, C150.2, C151.2, C152.2, C153.2, C154.2, C155.2, C156.2, C157.2, C158.2, C159.2, C160.2, C161.2, C162.2, C163.2, C164.2, C165.2, R102.2, U101.1 (GND), U101.9 (GND)
- net GPIO0: now also U102.L18 (IO_L4N_T0_D05_14)
- net GPIO1: now also U102.K18 (IO_L3N_T0_DQS_EMCCLK_14)
- net GPIO2: now also U102.J18 (IO_L3P_T0_DQS_PUDC_B_14)
- net GPIO3: now also U102.H18 (IO_L23N_T3_FWE_B_15)
- net GPIO4: now also U102.C18 (IO_L18N_T2_A23_15)
- net GPIO5: now also U102.D18 (IO_L17N_T2_A25_15)
- net GPIO6: now also U102.E18 (IO_L24N_T3_RS0_15)
- net GPIO7: now also U102.F18 (IO_L19N_T3_A21_VREF_15)
- net JTAG_TCK: now also U102.F8 (TCK_0)
- net JTAG_TDI: now also U102.T9 (TDI_0)
- net JTAG_TDO: now also U102.T8 (TDO_0)
- net JTAG_TMS: now also U102.R8 (TMS_0)
- net LED1: now also U102.N18 (IO_L10P_T1_D14_14)
- net LED2: now also U102.P18 (IO_L10N_T1_D15_14)
- net LED3: now also U102.R18 (IO_L15P_T2_DQS_RDWR_B_14)
- net LED4: now also U102.T18 (IO_L15N_T2_DQS_DOUT_CSO_B_14)
- net MAIN_PWR: now also C102.1, U101.2 (VIN)
- net PCIE_RX0+: now also U102.E4 (MGTPRXP0_216)
- net PCIE_RX0-: now also U102.E3 (MGTPRXN0_216)
- net PCIE_TX0+: now also U102.H2 (MGTPTXP0_216)
- net PCIE_TX0-: now also U102.H1 (MGTPTXN0_216)
- net REFCLK+: now also U102.D6 (MGTREFCLK0P_216)
- net REFCLK-: now also U102.D5 (MGTREFCLK0N_216)
- net PCIE_RX0_PRE-: now reaches C118.2, J103.B15 (PETn0)
- net at U108.4 (PG), U109.3 (EN): now also U101.3 (EN)
- net REFCLK_PRE-: now reaches C116.2, J103.A14 (REFCLK-)
- net PCIE_TX0_PRE-: now reaches C120.1, J103.A17 (PERn0)
- net REFCLK_PRE+: now reaches C115.2, J103.A13 (REFCLK+)
- net PCIE_RX0_PRE+: now reaches C117.2, J103.B14 (PETp0)
- net PCIE_TX0_PRE+: now reaches C119.1, J103.A16 (PERp0)
- net MGTAVTT: now reaches U102.A2 (MGTAVTT)
- net MGTAVTT: now also U102.C1 (MGTAVTT), U102.E1 (MGTAVTT), U102.F3 (MGTAVTT), U102.G2 (MGTAVTT), C114.1, C134.1, C135.1, C140.1, C141.1, C142.1, L103.1
- net at U102.A6 (MGTRREF_216): now also R103.2
- net MGTAVCC: now reaches U102.B4 (MGTAVCC)
- net MGTAVCC: now also U102.C5 (MGTAVCC), U102.E5 (MGTAVCC), U102.F5 (MGTAVCC), C113.1, C133.1, C136.1, C137.1, C138.1, L102.2
- new net: R101.2, R102.1, U101.5 (FB)
- new net: C101.1, U101.7 (BOOT)
- new net: C101.2, L101.1, U101.8 (SW)
- new net: C104.1, U101.6 (VCC)
- new net +1V2: C103.1, L101.2, L103.2, R101.1, R103.1
- no-connect marks 42 -> 181
Other:
- note added: "Vout = 1.22"
- moved on the sheet: C105, C106, C107, C108, C109, C110, C111, C112, C115, C116, C117, C118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
